File: file5AC1BF71.sch (KiCad schematic (older format))
At the start: 20 parts

Commit message: schematic design update
Added clean signal input and selector switch (dirty signal will always go to mixer)
Changed lines of the file:
@@
 Connection ~ 9425 3425
 Wire Wire Line
-	9175 3425 9425 3425
-Wire Wire Line
-	9425 3425 9500 3425
+	9175 3425 9500 3425
 Wire Wire Line
 	9500 3225 9450 3225
@@
 Connection ~ 10200 3325
 Wire Wire Line
-	10100 3325 10200 3325
-Wire Wire Line
-	10200 3325 10300 3325
+	10100 3325 10300 3325
 Wire Wire Line
 	10200 4075 10200 3325
@@
 	7050 4550 7050 4325
 Wire Wire Line
-	7050 4550 7275 4550
-Wire Wire Line
-	7275 4550 8000 4550
+	7050 4550 8000 4550
 Wire Wire Line
 	7025 3950 7275 3950
@@
 	7275 4050 6925 4050
 Wire Wire Line
-	6925 3925 6925 4050
-Wire Wire Line
-	5825 3925 6225 3925
-Wire Wire Line
-	6225 3925 6925 3925
+	6925 4050 6925 3925
+Wire Wire Line
+	6925 3925 5825 3925
 Connection ~ 7275 3950
 Wire Wire Line
-	3875 4125 3875 4325
-Wire Wire Line
-	3875 4325 3875 4400
+	3875 4125 3875 4400
 Wire Wire Line
 	3875 5025 3875 4700
@@
 	7275 4975 7275 5650
 Wire Wire Line
-	7275 4475 7275 4550
-Wire Wire Line
-	7275 4550 7275 4675
+	7275 4475 7275 4675
 Wire Wire Line
 	7275 3725 7175 3725
 Connection ~ 7275 4050
 Wire Wire Line
-	7275 3725 7275 3950
-Wire Wire Line
-	7275 3950 7275 4050
-Wire Wire Line
-	7275 4050 7275 4175
+	7275 3725 7275 4175
 Wire Wire Line
 	5825 3725 6875 3725
@@
 	1950 4625 1950 4725
 Wire Wire Line
-	2650 3525 3000 3525
-Wire Wire Line
-	3000 3525 3225 3525
+	2650 3525 3225 3525
 Wire Wire Line
 	3000 4175 3000 3525
 Wire Wire Line
-	2725 4175 2875 4175
-Wire Wire Line
-	2875 4175 3000 4175
+	2725 4175 3000 4175
 Connection ~ 1950 4175
 Wire Wire Line
@@
 	1950 3625 2050 3625
 Wire Wire Line
-	1950 3625 1950 4175
-Wire Wire Line
-	1950 4175 1950 4325
+	1950 3625 1950 4325
 $Comp
 L R R_OA_OUT_F1
@@
 	8700 3425 8875 3425
 Wire Wire Line
-	5825 3525 6000 3525
-Wire Wire Line
-	6000 3525 8300 3525
+	5825 3525 8300 3525
 Wire Wire Line
 	6000 3525 6000 2050
@@
 	6900 2925 6900 2150
 Wire Wire Line
-	6825 2150 6900 2150
-Wire Wire Line
-	6900 2150 7050 2150
+	6825 2150 7050 2150
 Wire Wire Line
 	6950 1800 7200 1800
@@
 GND
 Wire Wire Line
-	7050 2000 7175 2000
-Wire Wire Line
-	7175 2000 7200 2000
+	7050 2000 7200 2000
 Wire Wire Line
 	7050 2150 7050 2000
@@
 	7900 2925 7900 1900
 Wire Wire Line
-	7800 1900 7900 1900
-Wire Wire Line
-	7900 1900 8125 1900
+	7800 1900 8125 1900
 Wire Wire Line
 	8125 1900 8125 3325

Commit message: Final RevA Schematic
Parts:
- removed C_LPF2: 470nF, symbol C
- removed HOLD1: SW_SPST, symbol SW_SPST
- removed U_OA_SAW1, U_OA_SAW2: _TL071, symbol _TL071
- added C1_NEG2, C2_NEG2: 10uF, Capacitors_SMD:CP_Elec_4x5.3, symbol CP
- added C_HOLD1: 2.2uF, Capacitors_SMD:C_0805_HandSoldering, symbol CP
- added C_HOLD2: 10uF, Capacitors_SMD:C_0805_HandSoldering, symbol CP
- added J_AUX2MAIN_FX1, J_AUX2MAIN_PLL1, J_MAIN2AUX_FX1, J_MAIN2AUX_PLL1: Conn_01x04, Pin_Headers:Pin_Header_Straight_1x04_Pitch2.54mm, symbol Conn_01x04
- added J_AUX2MAIN_FXSW1, J_MAIN2AUX_FXSW1: Conn_01x06, Pin_Headers:Pin_Header_Straight_1x06_Pitch2.54mm, symbol Conn_01x06
- added R_SAW1: 2K7, Resistors_SMD:R_0805_HandSoldering, symbol R
- added R_SAW2: 1K, Resistors_SMD:R_0805_HandSoldering, symbol R
- added SW_HOLD1: SW_SPDT, custom_sw:SW_SPDT_W6.86MM_L12.7MM_P4.8MM_D2MM, symbol SW_SPDT
- added U_NEG2: _TC7662B, SMD_Packages:SOIC-8-N, symbol _TC7662B
- added U_SAW_OA1: _TL072, SMD_Packages:SOIC-8-N, symbol _TL072
- C_LPF1, C_SH1, C_SUSTAIN1: footprint (none) -> Capacitors_SMD:C_0805_HandSoldering
- C_SAW1: renamed from C_SAWINT1; footprint (none) -> Capacitors_SMD:C_0805_HandSoldering
- C_VCO1: value 10nF -> 22nF; footprint (none) -> Capacitors_SMD:C_0805_HandSoldering
- DAMPEN1, FMOD1, SWING1, TRIG1: footprint (none) -> Potentiometers:Potentiometer_Bourns_PTV09A-1_Horizontal
- R_OA_IN1, R_OA_OUT1, R_OA_OUT_F1: footprint (none) -> Resistors_SMD:R_0805_HandSoldering
- SW_WAVE1: footprint (none) -> custom_sw:SW_SPDT_W6.86MM_L12.7MM_P4.8MM_D2MM
- U_OAFX_IN1, U_OAFX_OUT1: footprint (none) -> SMD_Packages:SOIC-8-N
- U_PLL1: footprint (none) -> SMD_Packages:SO-16-N
Connections:
- net labels added: DAMP_P1_2, DAMP_P3, FMOD_P1, FMOD_P2_P3, HOLDSEL_P1, HOLDSEL_P2, HOLDSEL_P3, SWING_P2_1, SWING_P3, TRIG_P1_2, TRIG_P3, WAVESEL_P1, WAVESEL_P2, WAVESEL_P3
- wire segments 79 -> 161
- no-connect marks 13 -> 11
Other:
- note added: "FREQUENCY\nMOD POT"
- note added: "GAIN = 1.37"
- note added: "PLL DAMPEN\nCONTROL POT"
- note added: "PLL INPUT\nTRIGGER POT\n"
- note added: "PLL SAMPLE AND\nHOLD SEL SWITCH"
- note added: "PLL SQUARE/RAMP \nSELECTOR SWITCH"
- note added: "PLL SWING\nCONTROL POT"
- note removed: "smaller value \nimproves tracking"
- moved on the sheet: C_LPF1, C_SAW1, C_SH1, C_SUSTAIN1, C_VCO1, DAMPEN1, FMOD1, R_OA_IN1, R_OA_OUT1, R_OA_OUT_F1, SWING1, SW_WAVE1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
