File: _saved_GuitarPLLSynthEffect.sch (KiCad schematic (older format))
At the start: 36 parts

Commit message: Board Design Update RevA
Parts:
- C_OABY1, C_OABY2, C_OABY3, C_OABY4, C_OABY5, C_OABY6, C_PWRBY2: footprint (none) -> Capacitors_SMD:C_0805_HandSoldering
- C_PWRBY1: footprint Capacitors_SMD:CP_Elec_4x5.3 -> Capacitors_SMD:C_0805_HandSoldering
- R_LED1: footprint (none) -> Resistors_SMD:R_0805_HandSoldering
Changed lines of the file:
@@
 	1775 5250 1825 5250
 Wire Wire Line
-	1825 5050 1825 5250
-Wire Wire Line
-	1825 5250 1825 5500
+	1825 5050 1825 5500
 Wire Wire Line
 	1475 1600 1550 1600
@@
 	9950 5500 9950 5975
 Wire Wire Line
-	2050 1350 2050 1400
-Wire Wire Line
-	2050 1400 2050 1450
+	2050 1350 2050 1450
 Connection ~ 2050 1400
 Wire Wire Line
@@
 	5400 1900 5225 1900
 Wire Wire Line
-	3875 2050 4100 2050
-Wire Wire Line
-	4100 2050 4225 2050
+	3875 2050 4225 2050
 Wire Wire Line
 	4100 2125 4100 2050
@@
 	5075 4425 5075 3825
 Wire Wire Line
-	4975 3825 5075 3825
-Wire Wire Line
-	5075 3825 7475 3825
+	4975 3825 7475 3825
 Wire Wire Line
 	9275 4900 9275 5100
@@
 	8550 4700 9075 4700
 Wire Wire Line
-	8550 4700 8550 5250
-Wire Wire Line
-	8550 5250 8550 5375
+	8550 4700 8550 5375
 Wire Wire Line
 	8550 5250 9225 5250
@@
 	9775 5250 9775 4600
 Wire Wire Line
-	9675 4600 9775 4600
-Wire Wire Line
-	9775 4600 9950 4600
+	9675 4600 9950 4600
 Wire Wire Line
 	9950 4600 9950 5200
@@
 Connection ~ 5075 3825
 Wire Wire Line
-	7475 4250 7475 4950
-Wire Wire Line
-	7475 4950 7475 5650
+	7475 4250 7475 5650
 Wire Wire Line
 	4200 5175 3850 5175
@@
 	6200 5050 5550 5050
 Wire Wire Line
-	5550 5050 5550 5650
-Wire Wire Line
-	5550 5650 5550 5750
-Wire Wire Line
-	5550 5650 6475 5650
-Wire Wire Line
-	6475 5650 6775 5650
+	5550 5050 5550 5750
+Wire Wire Line
+	5550 5650 6775 5650
 Wire Wire Line
 	7475 5650 7000 5650
@@
 	3050 3725 4375 3725
 Wire Wire Line
-	3050 3375 3050 3725
-Wire Wire Line
-	3050 3725 3050 4750
+	3050 3375 3050 4750
 Wire Wire Line
 	3050 4750 3450 4750
@@
 	1775 3575 1850 3575
 Wire Wire Line
-	1850 3375 1850 3575
-Wire Wire Line
-	1850 3575 1850 3875
+	1850 3375 1850 3875
 Text Label 1850 3875 1    60   ~ 0
 GND
@@
 Optional clean signal for FX
 Wire Wire Line
-	1475 1400 2050 1400
-Wire Wire Line
-	2050 1400 2625 1400
-Wire Wire Line
-	2625 1400 3125 1400
-Wire Wire Line
-	3425 1400 3700 1400
-Wire Wire Line
-	3700 1400 4075 1400
-Wire Wire Line
-	4075 1400 5350 1400
+	1475 1400 3125 1400
+Wire Wire Line
+	3425 1400 5350 1400
 $Comp
 L _Schottky D_IN1
@@
 	1550 1600 1550 1825
 Wire Wire Line
-	1550 1825 2050 1825
-Wire Wire Line
-	2050 1825 2625 1825
-Wire Wire Line
-	2625 1825 2625 1825
-Wire Wire Line
-	2625 1825 2625 2100
+	1550 1825 2625 1825
+Wire Wire Line
+	2625 1750 2625 2100
 Wire Wire Line
 	2050 1750 2050 1825
@@
 F 0 "C_PWRBY1" H 2075 1700 50  0000 L CNN
 F 1 "10uF" H 2075 1500 50  0000 L CNN
-F 2 "Capacitors_SMD:CP_Elec_4x5.3" H 2088 1450 50  0001 C CNN
+F 2 "Capacitors_SMD:C_0805_HandSoldering" H 2088 1450 50  0001 C CNN
 F 3 "" H 2050 1600 50  0001 C CNN
 	1    2050 1600
@@
 	5100 7300 5100 7325
 Wire Wire Line
-	4875 7325 5100 7325
-Wire Wire Line
-	5100 7325 5275 7325
+	4875 7325 5275 7325
 Wire Wire Line
 	4875 7325 4875 7250
@@
 F 0 "R_LED1" V 2655 6475 50  0000 C CNN
 F 1 "2K7" V 2575 6475 50  0000 C CNN
-F 2 "" V 2505 6475 50  0001 C CNN
+F 2 "Resistors_SMD:R_0805_HandSoldering" V 2505 6475 50  0001 C CNN
 F 3 "" H 2575 6475 50  0001 C CNN
 	1    2575 6475
@@
 F 0 "C_OABY1" V 4025 3250 50  0000 L CNN
 F 1 "100nF" V 4100 3250 50  0000 L CNN
-F 2 "" H 4213 3375 50  0001 C CNN
+F 2 "Capacitors_SMD:C_0805_HandSoldering" H 4213 3375 50  0001 C CNN
 F 3 "" H 4175 3525 50  0001 C CNN
 	1    4175 3525
@@
 F 0 "C_OABY5" V 6000 4350 50  0000 L CNN
 F 1 "100nF" V 6075 4350 50  0000 L CNN
-F 2 "" H 6188 4500 50  0001 C CNN
+F 2 "Capacitors_SMD:C_0805_HandSoldering" H 6188 4500 50  0001 C CNN
 F 3 "" H 6150 4650 50  0001 C CNN
 	1    6150 4650
@@
 F 0 "C_OABY3" V 8725 4025 50  0000 L CNN
 F 1 "100nF" V 8800 4025 50  0000 L CNN
-F 2 "" H 8913 4150 50  0001 C CNN
+F 2 "Capacitors_SMD:C_0805_HandSoldering" H 8913 4150 50  0001 C CNN
 F 3 "" H 8875 4300 50  0001 C CNN
 	1    8875 4300
@@
 F 0 "C_OABY2" V 4200 3850 50  0000 L CNN
 F 1 "100nF" V 4275 3850 50  0000 L CNN
-F 2 "" H 4363 3975 50  0001 C CNN
+F 2 "Capacitors_SMD:C_0805_HandSoldering" H 4363 3975 50  0001 C CNN
 F 3 "" H 4325 4125 50  0001 C CNN
 	1    4325 4125
@@
 F 0 "C_OABY4" V 8925 4625 50  0000 L CNN
 F 1 "100nF" V 9000 4625 50  0000 L CNN
-F 2 "" H 9088 4750 50  0001 C CNN
+F 2 "Capacitors_SMD:C_0805_HandSoldering" H 9088 4750 50  0001 C CNN
 F 3 "" H 9050 4900 50  0001 C CNN
 	1    9050 4900
@@
 F 0 "C_OABY6" V 6050 4950 50  0000 L CNN
 F 1 "100nF" V 6125 4950 50  0000 L CNN
-F 2 "" H 6213 5100 50  0001 C CNN
+F 2 "Capacitors_SMD:C_0805_HandSoldering" H 6213 5100 50  0001 C CNN
 F 3 "" H 6175 5250 50  0001 C CNN
 	1    6175 5250
@@
 F 0 "C_PWRBY2" H 2225 1500 50  0000 L CNN
 F 1 "100nF" H 2375 1700 50  0000 L CNN
-F 2 "" H 2663 1450 50  0001 C CNN
+F 2 "Capacitors_SMD:C_0805_HandSoldering" H 2663 1450 50  0001 C CNN
 F 3 "" H 2625 1600 50  0001 C CNN
 	1    2625 1600
@@
 	2625 1450 2625 1400
 Connection ~ 2625 1400
-Wire Wire Line
-	2625 1750 2625 1825
 Connection ~ 2625 1825
 $EndSCHEMATC
